File: hardware/encoder.sch (EAGLE design)
At the start: 11 parts

Commit message: encoder brd
Parts:
- removed !CS, A, B, CLK, GND, MISO, MOSI, VCC: (no value), wirepad:SMD5
- added PAD2, PAD3, PAD4, PAD5, PAD6, PAD7, PAD8: (no value), wirepad:SMD2
Connections:
- removed net N$38: !CS.P, U$1.!CS
- removed net N$39: CLK.P, U$1.CLK
- removed net N$40: MISO.P, U$1.MISO
- removed net N$41: MOSI.P, U$1.MOSI
- removed net N$42: A.P, U$1.A
- removed net N$43: B.P, U$1.B
- removed net N$46: C5.1, U$1.VDD, U$1.VDD3V, VCC.P
- new net A: PAD6.P, U$1.A
- new net B: PAD7.P, U$1.B
- new net CLK: PAD2.P, U$1.CLK
- new net CS: PAD1.P, U$1.!CS
- new net MISO: PAD3.P, U$1.MISO
- new net MOSI: PAD4.P, U$1.MOSI
- new net VCC: C5.1, PAD8.P, U$1.VDD, U$1.VDD3V
- net GND: now also PAD5.P; no longer GND.P
Other:
- moved on the sheet: PAD1
Changed lines of the file:
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@@
 <part name="AGND30" library="supply2" deviceset="GND" device=""/>
 <part name="AGND31" library="supply2" deviceset="GND" device=""/>
-<part name="!CS" library="wirepad" deviceset="SMD5" device=""/>
-<part name="CLK" library="wirepad" deviceset="SMD5" device=""/>
-<part name="MISO" library="wirepad" deviceset="SMD5" device=""/>
-<part name="MOSI" library="wirepad" deviceset="SMD5" device=""/>
-<part name="A" library="wirepad" deviceset="SMD5" device=""/>
-<part name="B" library="wirepad" deviceset="SMD5" device=""/>
-<part name="VCC" library="wirepad" deviceset="SMD5" device=""/>
-<part name="GND" library="wirepad" deviceset="SMD5" device=""/>
 <part name="AGND1" library="supply2" deviceset="GND" device=""/>
 <part name="PAD1" library="wirepad" deviceset="SMD2" device=""/>
+<part name="PAD2" library="wirepad" deviceset="SMD2" device=""/>
+<part name="PAD3" library="wirepad" deviceset="SMD2" device=""/>
+<part name="PAD4" library="wirepad" deviceset="SMD2" device=""/>
+<part name="PAD8" library="wirepad" deviceset="SMD2" device=""/>
+<part name="PAD5" library="wirepad" deviceset="SMD2" device=""/>
+<part name="PAD6" library="wirepad" deviceset="SMD2" device=""/>
+<part name="PAD7" library="wirepad" deviceset="SMD2" device=""/>
 </parts>
 <sheets>
@@
 <instance part="AGND30" gate="GND" x="15.24" y="-12.7"/>
 <instance part="AGND31" gate="GND" x="-12.7" y="-12.7"/>
-<instance part="!CS" gate="1" x="-15.24" y="12.7" smashed="yes">
-<attribute name="NAME" x="-24.003" y="12.0142" size="1.778" layer="95"/>
-<attribute name="VALUE" x="-16.383" y="9.398" size="1.778" layer="96"/>
-</instance>
-<instance part="CLK" gate="1" x="-15.24" y="10.16" smashed="yes">
-<attribute name="NAME" x="-24.003" y="9.4742" size="1.778" layer="95"/>
-<attribute name="VALUE" x="-16.383" y="6.858" size="1.778" layer="96"/>
-</instance>
-<instance part="MISO" gate="1" x="-15.24" y="7.62" smashed="yes">
-<attribute name="NAME" x="-24.003" y="6.9342" size="1.778" layer="95"/>
-<attribute name="VALUE" x="-16.383" y="4.318" size="1.778" layer="96"/>
-</instance>
-<instance part="MOSI" gate="1" x="-15.24" y="5.08" smashed="yes">
-<attribute name="NAME" x="-24.003" y="4.3942" size="1.778" layer="95"/>
-<attribute name="VALUE" x="-16.383" y="1.778" size="1.778" layer="96"/>
-</instance>
-<instance part="A" gate="1" x="-15.24" y="0" smashed="yes">
-<attribute name="NAME" x="-18.923" y="-0.6858" size="1.778" layer="95"/>
-<attribute name="VALUE" x="-16.383" y="-3.302" size="1.778" layer="96"/>
-</instance>
-<instance part="B" gate="1" x="-15.24" y="-2.54" smashed="yes">
-<attribute name="NAME" x="-18.923" y="-3.2258" size="1.778" layer="95"/>
-<attribute name="VALUE" x="-16.383" y="-5.842" size="1.778" layer="96"/>
-</instance>
-<instance part="VCC" gate="1" x="35.56" y="12.7" smashed="yes" rot="R180">
-<attribute name="NAME" x="44.323" y="13.3858" size="1.778" layer="95" rot="R180"/>
-<attribute name="VALUE" x="36.703" y="16.002" size="1.778" layer="96" rot="R180"/>
-</instance>
-<instance part="GND" gate="1" x="35.56" y="10.16" smashed="yes" rot="R180">
-<attribute name="NAME" x="44.323" y="10.8458" size="1.778" layer="95" rot="R180"/>
-<attribute name="VALUE" x="36.703" y="13.462" size="1.778" layer="96" rot="R180"/>
-</instance>
 <instance part="AGND1" gate="GND" x="30.48" y="5.08"/>
-<instance part="PAD1" gate="1" x="-43.18" y="-7.62"/>
+<instance part="PAD1" gate="1" x="-15.24" y="12.7"/>
+<instance part="PAD2" gate="1" x="-15.24" y="10.16"/>
+<instance part="PAD3" gate="1" x="-15.24" y="7.62"/>
+<instance part="PAD4" gate="1" x="-15.24" y="5.08"/>
+<instance part="PAD8" gate="1" x="35.56" y="12.7" rot="R180"/>
+<instance part="PAD5" gate="1" x="35.56" y="10.16" rot="R180"/>
+<instance part="PAD6" gate="1" x="-15.24" y="0"/>
+<instance part="PAD7" gate="1" x="-15.24" y="-2.54"/>
 </instances>
 <busses>
@@
 </segment>
 <segment>
-<pinref part="GND" gate="1" pin="P"/>
-<wire x1="33.02" y1="10.16" x2="30.48" y2="10.16" width="0.1524" layer="91"/>
-<wire x1="30.48" y1="10.16" x2="30.48" y2="7.62" width="0.1524" layer="91"/>
 <pinref part="AGND1" gate="GND" pin="GND"/>
+<pinref part="PAD5" gate="1" pin="P"/>
+<wire x1="30.48" y1="7.62" x2="30.48" y2="10.16" width="0.1524" layer="91"/>
+<wire x1="30.48" y1="10.16" x2="33.02" y2="10.16" width="0.1524" layer="91"/>
 </segment>
 </net>
-<net name="N$38" class="0">
+<net name="CS" class="0">
 <segment>
 <pinref part="U$1" gate="G$1" pin="!CS"/>
 <wire x1="-10.16" y1="12.7" x2="-12.7" y2="12.7" width="0.1524" layer="91"/>
-<pinref part="!CS" gate="1" pin="P"/>
+<pinref part="PAD1" gate="1" pin="P"/>
 </segment>
 </net>
-<net name="N$39" class="0">
+<net name="CLK" class="0">
 <segment>
 <pinref part="U$1" gate="G$1" pin="CLK"/>
 <wire x1="-10.16" y1="10.16" x2="-12.7" y2="10.16" width="0.1524" layer="91"/>
-<pinref part="CLK" gate="1" pin="P"/>
+<pinref part="PAD2" gate="1" pin="P"/>
 </segment>
 </net>
-<net name="N$40" class="0">
+<net name="MISO" class="0">
 <segment>
 <pinref part="U$1" gate="G$1" pin="MISO"/>
 <wire x1="-10.16" y1="7.62" x2="-12.7" y2="7.62" width="0.1524" layer="91"/>
-<pinref part="MISO" gate="1" pin="P"/>
+<pinref part="PAD3" gate="1" pin="P"/>
 </segment>
 </net>
-<net name="N$41" class="0">
+<net name="MOSI" class="0">
 <segment>
 <pinref part="U$1" gate="G$1" pin="MOSI"/>
 <wire x1="-10.16" y1="5.08" x2="-12.7" y2="5.08" width="0.1524" layer="91"/>
-<pinref part="MOSI" gate="1" pin="P"/>
+<pinref part="PAD4" gate="1" pin="P"/>
 </segment>
 </net>
-<net name="N$42" class="0">
+<net name="A" class="0">
 <segment>
 <pinref part="U$1" gate="G$1" pin="A"/>
 <wire x1="-10.16" y1="0" x2="-12.7" y2="0" width="0.1524" layer="91"/>
-<pinref part="A" gate="1" pin="P"/>
+<pinref part="PAD6" gate="1" pin="P"/>
 </segment>
 </net>
-<net name="N$43" class="0">
+<net name="B" class="0">
 <segment>
 <pinref part="U$1" gate="G$1" pin="B"/>
 <wire x1="-10.16" y1="-2.54" x2="-12.7" y2="-2.54" width="0.1524" layer="91"/>
-<pinref part="B" gate="1" pin="P"/>
+<pinref part="PAD7" gate="1" pin="P"/>
 </segment>
 </net>
-<net name="N$46" class="0">
+<net name="VCC" class="0">
 <segment>
 <pinref part="U$1" gate="G$1" pin="VDD"/>
@@
 <wire x1="15.24" y1="12.7" x2="20.32" y2="12.7" width="0.1524" layer="91"/>
 <wire x1="20.32" y1="12.7" x2="20.32" y2="10.16" width="0.1524" layer="91"/>
-<pinref part="VCC" gate="1" pin="P"/>
-<wire x1="20.32" y1="12.7" x2="33.02" y2="12.7" width="0.1524" layer="91"/>
+<pinref part="PAD8" gate="1" pin="P"/>
+<wire x1="33.02" y1="12.7" x2="20.32" y2="12.7" width="0.1524" layer="91"/>
 <junction x="20.32" y="12.7"/>
 </segment>
