File: hardware/main.brd (EAGLE design)
At the start: 95.2 x 80.4 mm, 104 parts, among them IC1 MPU-6050, IC2 TB6612FNG, M1 MOTOR_MOUNT_V2, M2 LED_MOUNT, M3 LED_MOUNT, M4 LED_MOUNT, M5 LED_MOUNT, M6 LED_MOUNT, M7 LED_MOUNT, Q7 IRLML2244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

Commit message: Rozmieszczone diody na dziobie, przelotki przy DCDC
Parts:
- removed R10, R13, R15, R17, R6, R8: 10k, rcl:R0603
- removed T1: IRLML0030, zetex:SOT-23
- added T7: IRLML0030, zetex:SOT-23
- moved R12 177.5 mm to (57.1, -28.4), turned to 0 degrees
- moved R16 168.8 mm to (54.4, 28.8), turned to 90 degrees
- moved T4 149.4 mm to (53.5, -21.8), turned to 180 degrees
- moved R14 135.5 mm to (59.8, 28.8), turned to 90 degrees
- moved R5 135.3 mm to (57.1, 28.8), turned to 90 degrees
- moved T3 101.2 mm to (56.0, 24.9), turned to 180 degrees
- moved R7 100.2 mm to (53.7, -28.4), turned to 0 degrees
- moved T2 99.1 mm to (49.1, 24.9), turned to 180 degrees
- moved R9 97.1 mm to (56.8, -25.4)
- moved M7 70.0 mm to (63.0, -35.0)
- moved M3 56.5 mm to (85.7, 16.7), turned to 40 degrees
- moved T6 53.4 mm to (52.6, 24.9), turned to 180 degrees
- moved R29 39.1 mm to (73.8, -29.4), turned to 225 degrees
- moved M2 38.8 mm to (63.0, 35.0), turned to 0 degrees
- moved R33 33.5 mm to (74.8, 28.2), turned to 315 degrees
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- renumbered U$1 to ON
Connections:
- net ADC_L: now also M3.E, R3.2; no longer M7.E, R4.2
- net ADC_LF: now also R4.2, U$6.PA3; no longer R23.2, U$6.PA2
- net ADC_LS: now also M6.E, R23.2, U$6.PA2; no longer M3.E, R24.2, U$6.PA3
- net ADC_R: now also M4.E, R1.2; no longer M6.E, R3.2
- net ADC_RF: now also M7.E, R24.2; no longer M5.E, R2.2
- net ADC_RS: now also M5.E, R2.2; no longer M4.E, R1.2
- net D_L: now also T3.3; no longer R6.2, T1.3
- net D_LF: now also T2.3, T6.3; no longer R15.2, T5.3
- net D_LS: no longer R10.2, T3.3
- net D_R: now also T4.3, U$6.PC15; no longer R8.2, T2.3, U$6.PC13
- net D_RF: now also T7.3, U$6.PC13; no longer R17.2, T6.3, U$6.PC14
- net D_RS: now also T5.3, U$6.PC14; no longer R13.2, T4.3, U$6.PC15
- net GND: now also T7.2; no longer R10.1, R13.1, R15.1, R17.1, R6.1, R8.1, T1.2
- net N$1: now also M7.-; no longer M3.-
- net N$10: now also M3.-; no longer M6.-
- net N$11: now also T3.1; no longer T5.1
- net N$12: now also M2.-; no longer M7.-
- net N$13: now also T2.1; no longer T6.1
- net N$3: now also M6.-; no longer M2.-
- net N$4: now also T6.1; no longer T1.1
- net N$5: now also T7.1; no longer T2.1
- net N$7: now also T4.1; no longer T3.1
- net N$9: now also T5.1; no longer T4.1
Routing:
- net VCC: track 18.3 -> 163.4 mm, vias 2 -> 3
- net ADC_LS: track 13.0 -> 83.2 mm, vias 2 -> 1
- net N$3: track 0.00 -> 60.6 mm
- net ADC_RS: track 21.0 -> 80.7 mm
- net N$8: track 0.00 -> 55.2 mm
- net +3V3: track 289.6 -> 344.3 mm
- net ADC_L: track 21.0 -> 69.7 mm, vias 0 -> 1
- net ADC_R: track 24.1 -> 71.9 mm, vias 0 -> 1
- net N$6: track 0.00 -> 41.7 mm
- net N$10: track 0.00 -> 39.5 mm
- net ADC_LF: track 14.0 -> 40.3 mm, vias 2 -> 1
- net GND: track 0.00 -> 18.8 mm, vias 8 -> 36
- net ADC_RF: track 22.3 -> 37.0 mm
- net D_LF: track 16.8 -> 25.8 mm
- net N$1: track 0.00 -> 8.41 mm
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
Commit message: merge hardware_develTemp into hardware_devel
Parts:
- moved R12 1.55 mm to (56.9, -26.9), turned to 315 degrees
- moved R9 1.20 mm to (57.9, -25.0), turned to 315 degrees
- moved T5 1.20 mm to (54.6, -24.8)
- moved T7 1.13 mm to (50.4, -24.5)
- moved T4 1.02 mm to (53.3, -20.8)
- moved R7 0.28 mm to (53.8, -28.2), turned to 315 degrees
Routing:
- net +3V3: track 344.3 -> 395.5 mm
- net N$1: track 8.41 -> 0.00 mm
- net GND: track 18.8 -> 12.0 mm
- net N$9: track 3.77 -> 1.86 mm
- net N$6: track 41.7 -> 40.2 mm
- net D_R: track 23.2 -> 22.1 mm
- net N$7: track 5.56 -> 6.50 mm
- net N$8: track 55.2 -> 56.1 mm
- net D_RF: track 25.5 -> 24.7 mm
- net ENCL_A: track 51.7 -> 52.2 mm
Other:
- outline, holes or cut-outs redrawn

Commit message: 3d model - v1, gnd plane fun
Parts:
- removed LED6: blue, led:SML1206
- removed R33: 33R, resistor:R0805
- removed S2: (no value), EAGLE-TACT_SWITCHES-rev17c:450301014042
- moved R24 166.8 mm to (56.7, -31.3), turned to 315 degrees
- moved R23 113.3 mm to (84.7, 9.27), turned to 45 degrees
- moved R2 111.4 mm to (84.6, -8.89), turned to 0 degrees
- moved R1 109.6 mm to (82.7, -20.1), turned to 135 degrees
- moved R4 103.9 mm to (59.1, 30.9), turned to 0 degrees
- moved R3 93.0 mm to (82.2, 19.4), turned to 180 degrees
- moved R29 35.8 mm to (93.7, 0.39), turned to 270 degrees
- moved LED4 29.3 mm to (91.6, 0.13), turned to 90 degrees
- moved T2 3.90 mm to (53.0, 25.5), turned to 90 degrees
- moved R5 3.82 mm to (53.3, 28.6), turned to 45 degrees
- moved T6 3.49 mm to (49.1, 25.5), turned to 90 degrees
- moved R14 2.95 mm to (57.5, 27.0), turned to 45 degrees
- moved R16 1.50 mm to (55.3, 27.7), turned to 45 degrees
- moved R9 1.24 mm to (57.7, -26.2)
- moved M3 1.17 mm to (86.6, 16.0)
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Connections:
- removed net LED5: LED6.C
- removed net N$25: LED6.A, R33.1
- removed net N$3: M6.-, R5.2
- removed net OSC_IN: U$6.PH0
- new net N$2: M2.-, R5.2
- net +3V3: no longer R33.2
- net ADC_RF: now also U$6.PC0; no longer U$6.PC1
- net ADC_RS: now also U$6.PC1; no longer U$6.PC0
- net D_LF: now also U$6.PA6; no longer T2.3, U$6.PA5
- net D_LS: now also T2.3, U$6.PA5; no longer U$6.PA6
- net LED4: now also U$6.PH0
- net N$12: now also M6.-; no longer M2.-
Routing:
- net +3V3: track 395.5 -> 510.9 mm, vias 8 -> 12
- net LED4: track 0.00 -> 92.4 mm
- net N$3: track 60.6 -> 0.00 mm
- net N$12: track 4.80 -> 56.0 mm
- net VCC: track 163.4 -> 203.1 mm
- net GNDA: track 0.00 -> 9.93 mm, vias 0 -> 4
- net N$1: track 0.00 -> 8.35 mm
- net GND: track 12.0 -> 19.1 mm, vias 36 -> 65
- net N$2: track 0.00 -> 5.56 mm
- net D_LF: track 25.8 -> 30.6 mm
- net N$13: track 6.09 -> 1.87 mm
- net ADC_RS: track 80.7 -> 84.4 mm, vias 0 -> 2
- net +7V: track 88.7 -> 91.5 mm
- net VCAP_1: track 0.00 -> 2.67 mm
- net N$11: track 4.69 -> 2.04 mm
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- added copper zone on layer 1, net AGND
- added copper zone on layer 16, net AGND
- added copper zone on layer 1, net GNDA
- added copper zone on layer 16, net GNDA
Other:
- outline, holes or cut-outs redrawn

Commit message: almost done, gnd mess
Parts:
- moved M3 1.08 mm to (85.8, 16.7), turned to 50 degrees
- moved T4 0.74 mm to (53.3, -21.6)
- moved C1 0.13 mm to (57.4, 4.32)
- moved C25 0.13 mm to (55.4, 4.32)
Routing:
- net GND: track 19.1 -> 27.7 mm, vias 65 -> 73
- net +7V: track 91.5 -> 98.0 mm
- net +3V3: track 510.9 -> 515.2 mm
- net N$7: track 8.79 -> 7.52 mm
- net ADC_LS: track 85.4 -> 86.1 mm
- net D_R: track 22.1 -> 22.8 mm
- net D_RS: track 23.7 -> 24.4 mm
- net ENCL_A: track 52.2 -> 51.7 mm
- net D_LS: track 29.3 -> 29.9 mm

Commit message: led resistors changed to 0603, fixed gnd plane
Parts:
- R22, R25, R26, R27, R28, R29, R32: device resistor:R0805 -> resistor:R0603
- moved R22 0.16 mm to (17.1, -16.9)
- moved R32 0.13 mm to (21.8, -19.7)
Routing:
- net GND: track 27.7 -> 26.6 mm, vias 73 -> 82

Commit message: polygons fix
Parts:
- added U$1: GND_CONN, micromouse:GND_CONN
Connections:
- net GND: now also U$1.AGND, U$1.ANGD1
- net GNDA: now also U$1.GND, U$1.GND1
Routing:
- net +3V3: track 515.4 -> 514.5 mm
- net GND: vias 82 -> 83
Changed lines of the file:
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@@
 <element name="M2" library="micromouse" package="LED_MOUNT" value="LED_MOUNT" x="63" y="35"/>
 <element name="L1" library="micromouse" package="LABIRYNT" value="LABITYNT" x="28" y="0" rot="R270"/>
+<element name="U$1" library="micromouse" package="GND_CONN" value="GND_CONN" x="10.3124" y="3.2766" rot="R90"/>
 </elements>
 <signals>
@@
 <via x="19.2786" y="-12.0904" extent="1-16" drill="0.3"/>
 <via x="18.0086" y="-10.9474" extent="1-16" drill="0.3"/>
-<polygon width="0.3048" layer="1" isolate="0.3048" rank="6">
+<polygon width="0.3048" layer="1" isolate="0.3048" rank="4">
 <vertex x="51.435" y="-9.906"/>
 <vertex x="35.814" y="-9.906"/>
@@
 <via x="44.577" y="14.224" extent="1-16" drill="0.3"/>
 <via x="45.085" y="22.987" extent="1-16" drill="0.3"/>
-<polygon width="0.254" layer="1" isolate="0.3048">
+<polygon width="0.254" layer="1" isolate="0.3048" rank="3">
 <vertex x="56.261" y="-10.922"/>
 <vertex x="60.198" y="-6.35"/>
@@
 <vertex x="54.864" y="10.541"/>
 <vertex x="54.864" y="6.604"/>
-<vertex x="53.467" y="6.604"/>
-<vertex x="53.467" y="1.905"/>
-<vertex x="53.086" y="1.524"/>
+<vertex x="53.848" y="6.604"/>
+<vertex x="53.848" y="2.413"/>
+<vertex x="52.959" y="1.524"/>
 <vertex x="50.927" y="1.524"/>
 <vertex x="50.927" y="-4.318"/>
@@
 <via x="42.8244" y="-2.1336" extent="1-16" drill="0.3"/>
 <via x="39.9542" y="-0.127" extent="1-16" drill="0.3"/>
-<polygon width="0.3048" layer="16" isolate="0.3048" rank="6">
+<polygon width="0.3048" layer="16" isolate="0.3048" rank="4">
 <vertex x="51.435" y="-9.906"/>
 <vertex x="35.814" y="-9.906"/>
@@
 <vertex x="-0.508" y="25.654"/>
 <vertex x="2.413" y="28.575"/>
-<vertex x="52.07" y="28.575"/>
-<vertex x="52.197" y="11.049"/>
-<vertex x="50.546" y="9.144"/>
-<vertex x="48.133" y="9.144"/>
+<vertex x="52.324" y="28.575"/>
+<vertex x="52.324" y="11.176"/>
+<vertex x="50.3936" y="9.271"/>
+<vertex x="48.133" y="9.271"/>
 <vertex x="48.133" y="7.112"/>
 <vertex x="43.942" y="2.921"/>
@@
 <vertex x="36.322" y="-21.971"/>
 </polygon>
-<polygon width="0.254" layer="16" isolate="0.3048">
+<polygon width="0.254" layer="16" isolate="0.3048" rank="3">
 <vertex x="56.261" y="-10.922"/>
 <vertex x="60.198" y="-6.35"/>
@@
 <vertex x="54.864" y="10.541"/>
 <vertex x="54.864" y="6.604"/>
-<vertex x="53.467" y="6.604"/>
-<vertex x="53.467" y="1.905"/>
-<vertex x="53.086" y="1.524"/>
+<vertex x="53.848" y="6.604"/>
+<vertex x="53.848" y="2.413"/>
+<vertex x="52.959" y="1.524"/>
 <vertex x="50.927" y="1.524"/>
 <vertex x="50.927" y="-4.318"/>
@@
 <via x="7.366" y="-0.635" extent="1-16" drill="0.3"/>
 <via x="39.9034" y="-25.6286" extent="1-16" drill="0.3"/>
+<via x="56.4134" y="-7.4676" extent="1-16" drill="0.3"/>
+<contactref element="U$1" pad="AGND"/>
+<contactref element="U$1" pad="ANGD1"/>
 </signal>
 <signal name="D_LS">
@@
 <wire x1="35.052" y1="5.588" x2="35.052" y2="11.303" width="0.4064" layer="16"/>
 <via x="35.052" y="11.303" extent="1-16" drill="0.3"/>
-<wire x1="35.052" y1="11.303" x2="35.052" y2="15.113" width="0.4064" layer="1"/>
-<wire x1="35.052" y1="15.113" x2="35.687" y2="15.748" width="0.4064" layer="1"/>
-<wire x1="35.687" y1="15.748" x2="40.005" y2="15.748" width="0.4064" layer="1"/>
+<wire x1="35.052" y1="11.303" x2="35.052" y2="15.748" width="0.4064" layer="1"/>
+<wire x1="34.29" y1="15.748" x2="35.052" y2="15.748" width="0.4064" layer="1"/>
+<wire x1="35.179" y1="15.748" x2="40.005" y2="15.748" width="0.4064" layer="1"/>
 <wire x1="40.005" y1="15.748" x2="40.386" y2="16.129" width="0.4064" layer="1"/>
 <wire x1="40.386" y1="16.129" x2="40.767" y2="16.51" width="0.4064" layer="1"/>
@@
 <wire x1="32.258" y1="26.162" x2="32.258" y2="17.78" width="0.4064" layer="1"/>
 <wire x1="32.258" y1="17.78" x2="34.29" y2="15.748" width="0.4064" layer="1"/>
-<wire x1="34.29" y1="15.748" x2="35.687" y2="15.748" width="0.4064" layer="1"/>
 <wire x1="5.207" y1="-21.336" x2="4.596" y2="-20.725" width="0.3048" layer="1"/>
 <wire x1="4.596" y1="-20.725" x2="4.596" y2="-20.156" width="0.3048" layer="1"/>
@@
 <wire x1="10.16" y1="22.606" x2="10.16" y2="24.257" width="0.4064" layer="1"/>
 <wire x1="7.749" y1="20.068" x2="6.729" y2="19.048" width="0.4064" layer="1"/>
-<wire x1="57.9092" y1="-36.2126" x2="59.2988" y2="-37.6022" width="0.4064" layer="1"/>
-<wire x1="59.2988" y1="-37.6022" x2="59.4156" y2="-37.719" width="0.4064" layer="1"/>
-<wire x1="59.4156" y1="-37.719" x2="65.913" y2="-37.719" width="0.4064" layer="1"/>
+<wire x1="55.118" y1="-37.719" x2="57.9092" y2="-37.719" width="0.4064" layer="1"/>
+<wire x1="57.9092" y1="-37.719" x2="65.913" y2="-37.719" width="0.4064" layer="1"/>
 <wire x1="70.231" y1="-33.401" x2="73.787" y2="-33.401" width="0.4064" layer="1"/>
 <wire x1="73.787" y1="-33.401" x2="90.424" y2="-16.764" width="0.4064" layer="1"/>
@@
 <wire x1="23.876" y1="-25.019" x2="30.734" y2="-25.019" width="0.4064" layer="1"/>
 <wire x1="30.734" y1="-25.019" x2="32.4612" y2="-26.7462" width="0.4064" layer="1"/>
-<wire x1="54.3052" y1="-36.9062" x2="55.245" y2="-37.846" width="0.4064" layer="1"/>
-<wire x1="55.245" y1="-37.846" x2="59.055" y2="-37.846" width="0.4064" layer="1"/>
-<wire x1="59.055" y1="-37.846" x2="59.2988" y2="-37.6022" width="0.4064" layer="1" curve="90"/>
 <wire x1="16.129" y1="-24.638" x2="18.923" y2="-21.844" width="0.3048" layer="1"/>
 <wire x1="65.913" y1="-37.719" x2="70.231" y2="-33.401" width="0.4064" layer="1"/>
@@
 <wire x1="6.729" y1="19.048" x2="4.3368" y2="19.048" width="0.4064" layer="1"/>
 <wire x1="4.3368" y1="19.048" x2="4.3368" y2="19.021" width="0.4064" layer="1"/>
+<wire x1="54.3052" y1="-36.9062" x2="55.118" y2="-37.719" width="0.4064" layer="1"/>
+<wire x1="57.9092" y1="-36.2126" x2="57.9092" y2="-37.719" width="0.4064" layer="1"/>
+<wire x1="35.052" y1="15.748" x2="35.179" y2="15.748" width="0.4064" layer="1"/>
 <wire x1="13.94" y1="11.608" x2="13.942440625" y2="11.608659375" width="0" layer="19" extent="1-16"/>
 <wire x1="8.013559375" y1="-11.640659375" x2="8.016" y2="-11.64" width="0" layer="19" extent="1-16"/>
@@
 <contactref element="C6" pad="1"/>
 <contactref element="D9" pad="2"/>
-<polygon width="0.3048" layer="1" isolate="0.3048" rank="4">
+<polygon width="0.3048" layer="1" isolate="0.3048" rank="3">
 <vertex x="9.398" y="-3.556"/>
 <vertex x="14.351" y="-3.556"/>
@@
 <wire x1="10.6716" y1="-2.415" x2="10.2864" y2="-2.415" width="0.6096" layer="1"/>
 <wire x1="10.2864" y1="-2.415" x2="10.2864" y2="-0.251" width="0.6096" layer="1"/>
-<polygon width="0.3048" layer="16" isolate="0.3048" rank="4">
+<polygon width="0.3048" layer="16" isolate="0.3048" rank="3">
 <vertex x="9.398" y="-3.556"/>
 <vertex x="14.351" y="-3.556"/>
@@
 <wire x1="25.0444" y1="4.1656" x2="25.8826" y2="4.1656" width="0.3048" layer="1"/>
 <via x="10.287" y="-1.524" extent="1-16" drill="0.3"/>
+<contactref element="U$1" pad="GND"/>
+<contactref element="U$1" pad="GND1"/>
+<wire x1="10.3124" y1="2.6416" x2="10.3124" y2="2.6416" width="0" layer="19" extent="1-16"/>
 </signal>
 <signal name="N$38">
@@
 <contactref element="U$6" pad="VSSA"/>
 <contactref element="R1" pad="1"/>
-<polygon width="0.254" layer="1">
+<polygon width="0.254" layer="1" rank="4">
 <vertex x="51.435" y="-41.783"/>
 <vertex x="69.088" y="-41.783"/>
@@
 <via x="60.325" y="36.1442" extent="1-16" drill="0.3"/>
 <via x="72.2884" y="34.9504" extent="1-16" drill="0.3"/>
-<polygon width="0.254" layer="16">
+<polygon width="0.254" layer="16" rank="4">
 <vertex x="51.435" y="-41.783"/>
 <vertex x="69.088" y="-41.783"/>
@@
 <vertex x="54.229" y="-26.924"/>
 <vertex x="52.832" y="-26.924"/>
+<vertex x="52.451" y="-26.543"/>
+<vertex x="51.562" y="-26.543"/>
 <vertex x="51.435" y="-28.321"/>
 </polygon>
