File: hardware/encoder.brd (EAGLE design)
At the start: 30.5 x 21.3 mm, 11 parts

Commit message: encoder brd
Parts:
- removed !CS, A, B, CLK, GND, MISO, MOSI, VCC: (no value), wirepad:SMD2,54-5,08
- added PAD2, PAD3, PAD4, PAD5, PAD6, PAD7, PAD8: (no value), wirepad:SMD1,27-2,54
- moved C5 8.87 mm to (6.67, 9.03), flipped to the bottom, turned to 90 degrees
- moved U$1 8.16 mm to (8.40, 8.50)
- moved PAD1 6.39 mm to (5.40, 1.30), turned to 180 degrees
Connections:
- removed net N$38: !CS.1, U$1.1
- removed net N$39: CLK.1, U$1.2
- removed net N$40: MISO.1, U$1.3
- removed net N$41: MOSI.1, U$1.4
- removed net N$42: A.1, U$1.7
- removed net N$43: B.1, U$1.6
- removed net N$46: C5.1, U$1.11, U$1.12, VCC.1
- new net A: PAD6.1, U$1.7
- new net B: PAD7.1, U$1.6
- new net CLK: PAD2.1, U$1.2
- new net CS: PAD1.1, U$1.1
- new net MISO: PAD3.1, U$1.3
- new net MOSI: PAD4.1, U$1.4
- new net VCC: C5.1, PAD8.1, U$1.11, U$1.12
- net GND: now also PAD5.1; no longer GND.1
Routing:
- net VCC: track 0.00 -> 13.1 mm, vias 0 -> 1
- net MOSI: track 0.00 -> 6.30 mm
- net MISO: track 0.00 -> 5.72 mm
- net A: track 0.00 -> 5.01 mm, vias 0 -> 1
- net CS: track 0.00 -> 4.74 mm
- net B: track 0.00 -> 4.72 mm, vias 0 -> 1
- net CLK: track 0.00 -> 4.41 mm
- added copper zone on layer 1, net GND
- added copper zone on layer 16, net GND
Other:
- board size 30.5 x 21.3 mm -> 8.8 x 12.8 mm

Commit message: poukladanie warstwy opisowej, dodanie przelotek - wersja finalna
Changed lines of the file:
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@@
 <layer number="25" name="tNames" color="7" fill="1" visible="yes" active="yes"/>
 <layer number="26" name="bNames" color="7" fill="1" visible="yes" active="yes"/>
-<layer number="27" name="tValues" color="7" fill="1" visible="yes" active="yes"/>
-<layer number="28" name="bValues" color="7" fill="1" visible="yes" active="yes"/>
+<layer number="27" name="tValues" color="7" fill="1" visible="no" active="yes"/>
+<layer number="28" name="bValues" color="7" fill="1" visible="no" active="yes"/>
 <layer number="29" name="tStop" color="7" fill="3" visible="no" active="yes"/>
 <layer number="30" name="bStop" color="7" fill="6" visible="no" active="yes"/>
@@
 <layer number="99" name="SpiceOrder" color="7" fill="1" visible="no" active="no"/>
 <layer number="100" name="Muster" color="7" fill="1" visible="no" active="no"/>
-<layer number="101" name="Patch_Top" color="12" fill="4" visible="yes" active="yes"/>
-<layer number="102" name="Vscore" color="7" fill="1" visible="yes" active="yes"/>
-<layer number="103" name="tMap" color="7" fill="1" visible="yes" active="yes"/>
-<layer number="104" name="Name" color="16" fill="1" visible="yes" active="yes"/>
-<layer number="105" name="tPlate" color="7" fill="1" visible="yes" active="yes"/>
-<layer number="106" name="bPlate" color="7" fill="1" visible="yes" active="yes"/>
-<layer number="107" name="Crop" color="7" fill="1" visible="yes" active="yes"/>
+<layer number="101" name="Patch_Top" color="12" fill="4" visible="no" active="yes"/>
+<layer number="102" name="Vscore" color="7" fill="1" visible="no" active="yes"/>
+<layer number="103" name="tMap" color="7" fill="1" visible="no" active="yes"/>
+<layer number="104" name="Name" color="16" fill="1" visible="no" active="yes"/>
+<layer number="105" name="tPlate" color="7" fill="1" visible="no" active="yes"/>
+<layer number="106" name="bPlate" color="7" fill="1" visible="no" active="yes"/>
+<layer number="107" name="Crop" color="7" fill="1" visible="no" active="yes"/>
 <layer number="108" name="fp8" color="7" fill="1" visible="no" active="yes"/>
 <layer number="109" name="fp9" color="7" fill="1" visible="no" active="yes"/>
@@
 </autorouter>
 <elements>
-<element name="C5" library="rcl" package="C0603" value="100n" x="6.67" y="9.0282" rot="MR90"/>
-<element name="U$1" library="ams" package="TSSOP-14" value="AS5147P" x="8.405" y="8.5" rot="R90"/>
-<element name="PAD1" library="wirepad" package="SMD1,27-2,54" value="" x="5.4" y="1.3" rot="R180"/>
-<element name="PAD2" library="wirepad" package="SMD1,27-2,54" value="" x="7.4" y="1.3" rot="R180"/>
-<element name="PAD3" library="wirepad" package="SMD1,27-2,54" value="" x="9.4" y="1.3" rot="R180"/>
-<element name="PAD4" library="wirepad" package="SMD1,27-2,54" value="" x="11.4" y="1.3" rot="R180"/>
-<element name="PAD8" library="wirepad" package="SMD1,27-2,54" value="" x="5.4" y="1.3" rot="MR0"/>
-<element name="PAD5" library="wirepad" package="SMD1,27-2,54" value="" x="7.402" y="1.298" rot="MR0"/>
-<element name="PAD6" library="wirepad" package="SMD1,27-2,54" value="" x="11.394" y="1.298" rot="MR0"/>
-<element name="PAD7" library="wirepad" package="SMD1,27-2,54" value="" x="9.396" y="1.298" rot="MR0"/>
+<element name="C5" library="rcl" package="C0603" value="100n" x="6.67" y="9.0282" smashed="yes" rot="MR90">
+<attribute name="NAME" x="8.305" y="7.3932" size="1.27" layer="26" rot="MR90"/>
+<attribute name="VALUE" x="4.765" y="8.3932" size="1.27" layer="28" rot="MR90"/>
+</element>
+<element name="U$1" library="ams" package="TSSOP-14" value="AS5147P" x="8.405" y="8.5" smashed="yes" rot="R90">
+<attribute name="VALUE" x="12.2912" y="6.4172" size="1.016" layer="27" ratio="10" rot="R90"/>
+</element>
+<element name="PAD1" library="wirepad" package="SMD1,27-2,54" value="" x="5.4" y="1.3" smashed="yes" rot="R180">
+<attribute name="VALUE" x="5.4" y="1.3" size="0.0254" layer="27" rot="R180"/>
+</element>
+<element name="PAD2" library="wirepad" package="SMD1,27-2,54" value="" x="7.4" y="1.3" smashed="yes" rot="R180">
+<attribute name="VALUE" x="7.4" y="1.3" size="0.0254" layer="27" rot="R180"/>
+</element>
+<element name="PAD3" library="wirepad" package="SMD1,27-2,54" value="" x="9.4" y="1.3" smashed="yes" rot="R180">
+<attribute name="VALUE" x="9.4" y="1.3" size="0.0254" layer="27" rot="R180"/>
+</element>
+<element name="PAD4" library="wirepad" package="SMD1,27-2,54" value="" x="11.4" y="1.3" smashed="yes" rot="R180">
+<attribute name="VALUE" x="11.4" y="1.3" size="0.0254" layer="27" rot="R180"/>
+</element>
+<element name="PAD8" library="wirepad" package="SMD1,27-2,54" value="" x="5.4" y="1.3" smashed="yes" rot="MR0">
+<attribute name="VALUE" x="5.4" y="1.3" size="0.0254" layer="28" rot="MR0"/>
+</element>
+<element name="PAD5" library="wirepad" package="SMD1,27-2,54" value="" x="7.402" y="1.298" smashed="yes" rot="MR0">
+<attribute name="VALUE" x="7.402" y="1.298" size="0.0254" layer="28" rot="MR0"/>
+</element>
+<element name="PAD6" library="wirepad" package="SMD1,27-2,54" value="" x="11.394" y="1.298" smashed="yes" rot="MR0">
+<attribute name="VALUE" x="11.394" y="1.298" size="0.0254" layer="28" rot="MR0"/>
+</element>
+<element name="PAD7" library="wirepad" package="SMD1,27-2,54" value="" x="9.396" y="1.298" smashed="yes" rot="MR0">
+<attribute name="VALUE" x="9.396" y="1.298" size="0.0254" layer="28" rot="MR0"/>
+</element>
 </elements>
 <signals>
